Commit message: changed mini 1.5 URDF file

File: mini_description/urdf/mini1.0/mini1.0_gazebo.urdf.xacro (robot description, xacro)
@@ -183,5 +183,5 @@
     <xacro:property name="min_angle" value="-180" />
     <xacro:property name="max_angle" value="180" /> -->
-    <gazebo reference="lidar_link">
+    <gazebo reference="laser_link">
       <sensor type="ray" name="lidar">
         <always_on>true</always_on>
@@ -209,5 +209,5 @@
           <updateRate>40</updateRate>
           <topicName>scan</topicName>
-          <frameName>base_laser_link</frameName>
+          <frameName>laser_link</frameName>
         </plugin>
       </sensor>

File: mini_description/urdf/mini1.5/god_arm_fore.urdf.xacro (robot description, xacro)
@@ -7,5 +7,5 @@
   <property name="arm_fore_radius" value="0.009" />
   <property name="arm_fore_length" value="0.18" />
-  <!-- Define the torso -->
+  <!-- Define the fore arm -->
   <macro name="arm_fore" params="parent name">
     <joint name="elbow_joint" type="revolute">
@@ -13,8 +13,8 @@
       <axis xyz="0 1 0"/>
       <limit effort="1.0" lower="${-M_PI/2}" upper="${M_PI/2}" velocity="1.571"/>
-      <parent link="${parent}_link"/>
-      <child link="${name}_link"/>
+      <parent link="arm_upper_link"/>
+      <child link="arm_fore_link"/>
     </joint>
-    <link name="${name}_link">
+    <link name="arm_fore_link">
       <inertial>
         <mass value="0.1" />

File: mini_description/urdf/mini1.5/god_arm_upper.urdf.xacro (robot description, xacro)
@@ -7,5 +7,5 @@
   <property name="arm_upper_radius" value="0.009" />
   <property name="arm_upper_length" value="0.4" />
-  <!-- Define the torso -->
+  <!-- Define the upper arm -->
   <macro name="arm_upper" params="parent name">
     <joint name="shoulder_joint" type="revolute">
@@ -13,8 +13,8 @@
       <axis xyz="0 1 0"/>
       <limit effort="1.0" lower="${-M_PI/2}" upper="0" velocity="1.571"/>
-      <parent link="${parent}_link"/>
-      <child link="${name}_link"/>
+      <parent link="torso_upper_link"/>
+      <child link="arm_upper_link"/>
     </joint>
-    <link name="${name}_link">
+    <link name="arm_upper_link">
       <inertial>
         <mass value="0.5" />

File: mini_description/urdf/mini1.5/mini1.5_gazebo.urdf.xacro (robot description, xacro)
@@ -183,5 +183,5 @@
     <xacro:property name="min_angle" value="-180" />
     <xacro:property name="max_angle" value="180" /> -->
-    <gazebo reference="lidar_link">
+    <gazebo reference="laser_link">
       <sensor type="ray" name="lidar">
         <always_on>true</always_on>
@@ -209,5 +209,5 @@
           <updateRate>40</updateRate>
           <topicName>scan</topicName>
-          <frameName>base_laser_link</frameName>
+          <frameName>laser_link</frameName>
         </plugin>
       </sensor>
